File: quad.kicad_sch (KiCad schematic)
At the start: 1 part, among them U2 PCAL6416AHF

Commit message: implement schematic review feedback
Parts:
- added C69, C71: 100n, Capacitor_SMD:C_0402_1005Metric, symbol Device:C
- renumbered U2 to U5
Connections:
- net +3V3: now also C71.1
- net GND: now also C69.2, C71.2
- net VIO: now also C69.1
Other:
- sheet SDI In 1 ports: added ~{VIO_GOOD}; removed none
- sheet SDI In 2 ports: added ~{VIO_GOOD}; removed none
- sheet SDI Out 1 ports: added VIO_GOOD; removed none
- sheet SDI Out 2 ports: added VIO_GOOD; removed none

Commit message: substitute bnc connector for better max freq
Parts:
- renumbered C69 to C40, C71 to C41
Changed lines of the file:
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@@
 		(dnp no)
 		(fields_autoplaced yes)
-		(property "Reference" "#PWR059"
+		(property "Reference" "#PWR063"
 			(at 83.82 66.04 0)
 			(hide yes)
@@
 			(project "syzygy-octosdi"
 				(path "/cb0cdcc9-6b9b-4b74-8146-9043de7999b1/7952d4e7-438b-4019-af07-2f77390b2cbe"
-					(reference "#PWR061")
-					(unit 1)
-				)
-				(path "/cb0cdcc9-6b9b-4b74-8146-9043de7999b1/86247bb6-a200-4434-96fd-e477d61cd494"
-					(reference "#PWR059")
+					(reference "#PWR068")
+					(unit 1)
+				)
+				(path "/cb0cdcc9-6b9b-4b74-8146-9043de7999b1/86247bb6-a200-4434-96fd-e477d61cd494"
+					(reference "#PWR063")
 					(unit 1)
 				)
@@
 		(dnp no)
 		(fields_autoplaced yes)
-		(property "Reference" "#PWR0125"
+		(property "Reference" "#PWR061"
 			(at 48.26 114.3 0)
 			(hide yes)
@@
 			(project "syzygy-octosdi"
 				(path "/cb0cdcc9-6b9b-4b74-8146-9043de7999b1/7952d4e7-438b-4019-af07-2f77390b2cbe"
-					(reference "#PWR0126")
-					(unit 1)
-				)
-				(path "/cb0cdcc9-6b9b-4b74-8146-9043de7999b1/86247bb6-a200-4434-96fd-e477d61cd494"
-					(reference "#PWR0125")
+					(reference "#PWR066")
+					(unit 1)
+				)
+				(path "/cb0cdcc9-6b9b-4b74-8146-9043de7999b1/86247bb6-a200-4434-96fd-e477d61cd494"
+					(reference "#PWR061")
 					(unit 1)
 				)
@@
 		(dnp no)
 		(fields_autoplaced yes)
-		(property "Reference" "#PWR058"
+		(property "Reference" "#PWR062"
 			(at 80.01 124.46 0)
 			(hide yes)
@@
 			(project "syzygy-octosdi"
 				(path "/cb0cdcc9-6b9b-4b74-8146-9043de7999b1/7952d4e7-438b-4019-af07-2f77390b2cbe"
-					(reference "#PWR060")
-					(unit 1)
-				)
-				(path "/cb0cdcc9-6b9b-4b74-8146-9043de7999b1/86247bb6-a200-4434-96fd-e477d61cd494"
-					(reference "#PWR058")
+					(reference "#PWR067")
+					(unit 1)
+				)
+				(path "/cb0cdcc9-6b9b-4b74-8146-9043de7999b1/86247bb6-a200-4434-96fd-e477d61cd494"
+					(reference "#PWR062")
 					(unit 1)
 				)
@@
 		(dnp no)
 		(fields_autoplaced yes)
-		(property "Reference" "C69"
+		(property "Reference" "C40"
 			(at 39.37 101.5999 0)
 			(show_name no)
@@
 			(project "syzygy-octosdi"
 				(path "/cb0cdcc9-6b9b-4b74-8146-9043de7999b1/7952d4e7-438b-4019-af07-2f77390b2cbe"
-					(reference "C70")
-					(unit 1)
-				)
-				(path "/cb0cdcc9-6b9b-4b74-8146-9043de7999b1/86247bb6-a200-4434-96fd-e477d61cd494"
-					(reference "C69")
+					(reference "C42")
+					(unit 1)
+				)
+				(path "/cb0cdcc9-6b9b-4b74-8146-9043de7999b1/86247bb6-a200-4434-96fd-e477d61cd494"
+					(reference "C40")
 					(unit 1)
 				)
@@
 		(dnp no)
 		(fields_autoplaced yes)
-		(property "Reference" "C71"
+		(property "Reference" "C41"
 			(at 52.07 101.5999 0)
 			(show_name no)
@@
 			(project "syzygy-octosdi"
 				(path "/cb0cdcc9-6b9b-4b74-8146-9043de7999b1/7952d4e7-438b-4019-af07-2f77390b2cbe"
-					(reference "C72")
-					(unit 1)
-				)
-				(path "/cb0cdcc9-6b9b-4b74-8146-9043de7999b1/86247bb6-a200-4434-96fd-e477d61cd494"
-					(reference "C71")
+					(reference "C43")
+					(unit 1)
+				)
+				(path "/cb0cdcc9-6b9b-4b74-8146-9043de7999b1/86247bb6-a200-4434-96fd-e477d61cd494"
+					(reference "C41")
 					(unit 1)
 				)
@@
 		(dnp no)
 		(fields_autoplaced yes)
-		(property "Reference" "#PWR0121"
+		(property "Reference" "#PWR060"
 			(at 48.26 101.6 0)
 			(hide yes)
@@
 			(project "syzygy-octosdi"
 				(path "/cb0cdcc9-6b9b-4b74-8146-9043de7999b1/7952d4e7-438b-4019-af07-2f77390b2cbe"
-					(reference "#PWR0122")
-					(unit 1)
-				)
-				(path "/cb0cdcc9-6b9b-4b74-8146-9043de7999b1/86247bb6-a200-4434-96fd-e477d61cd494"
-					(reference "#PWR0121")
+					(reference "#PWR065")
+					(unit 1)
+				)
+				(path "/cb0cdcc9-6b9b-4b74-8146-9043de7999b1/86247bb6-a200-4434-96fd-e477d61cd494"
+					(reference "#PWR060")
 					(unit 1)
 				)
@@
 		(dnp no)
 		(fields_autoplaced yes)
-		(property "Reference" "#PWR0123"
+		(property "Reference" "#PWR059"
 			(at 35.56 114.3 0)
 			(hide yes)
@@
 			(project "syzygy-octosdi"
 				(path "/cb0cdcc9-6b9b-4b74-8146-9043de7999b1/7952d4e7-438b-4019-af07-2f77390b2cbe"
-					(reference "#PWR0124")
-					(unit 1)
-				)
-				(path "/cb0cdcc9-6b9b-4b74-8146-9043de7999b1/86247bb6-a200-4434-96fd-e477d61cd494"
-					(reference "#PWR0123")
-					(unit 1)
-				)
+					(reference "#PWR064")
+					(unit 1)
+				)
+				(path "/cb0cdcc9-6b9b-4b74-8146-9043de7999b1/86247bb6-a200-4434-96fd-e477d61cd494"
+					(reference "#PWR059")
+					(unit 1)
+				)
