File: smartvio.kicad_sch (KiCad schematic)
At the start: 12 parts, among them J1 Conn_02x03_Odd_Even, U11 STM32G031G8Ux

Commit message: implement schematic review feedback
Parts:
- added D11: LED, LED_SMD:LED_0603_1608Metric, symbol Device:LED
- added R66, R67: 10k, Resistor_SMD:R_0603_1608Metric, symbol Device:R
- added R70: 4k7, Resistor_SMD:R_0603_1608Metric, symbol Device:R
- renumbered R41 to R63, R43 to R64, R45 to R65, TP2 to TP1, TP3 to TP2
Connections:
- net +3V3: now also R67.1
- net GND: now also D11.1 (K), R66.2
- net VIO: now reaches U11.7 (PA1)
- net VIO_GOOD: now reaches U11.8 (PA2)
- net VIO_GOOD: now also R66.1, R70.1
- net ~{VIO_GOOD}: now reaches U11.9 (PA3)
- net ~{VIO_GOOD}: now also R67.2
- new net: D11.2 (A), R70.2
- no-connect marks 17 -> 14

Commit message: substitute bnc connector for better max freq
Parts:
- renumbered C66 to C82, C67 to C83, C68 to C84, J1 to J9, R63 to R77, R64 to R78, R65 to R79, R67 to R80, R66 to R81, R70 to R82
Changed lines of the file:
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@@
 		(dnp no)
 		(fields_autoplaced yes)
-		(property "Reference" "#PWR016"
+		(property "Reference" "#PWR0128"
 			(at 162.56 138.43 0)
 			(hide yes)
@@
 			(project "syzygy-octosdi"
 				(path "/cb0cdcc9-6b9b-4b74-8146-9043de7999b1/731e7cbd-3c26-4319-8367-0b2702130274"
-					(reference "#PWR016")
+					(reference "#PWR0128")
 					(unit 1)
 				)
@@
 		(dnp no)
 		(fields_autoplaced yes)
-		(property "Reference" "C68"
+		(property "Reference" "C84"
 			(at 114.3 123.1962 0)
 			(show_name no)
@@
 			(project "syzygy-octosdi"
 				(path "/cb0cdcc9-6b9b-4b74-8146-9043de7999b1/731e7cbd-3c26-4319-8367-0b2702130274"
-					(reference "C68")
+					(reference "C84")
 					(unit 1)
 				)
@@
 		(in_pos_files yes)
 		(dnp no)
-		(property "Reference" "R67"
+		(property "Reference" "R80"
 			(at 135.89 128.2699 0)
 			(show_name no)
@@
 			(project "syzygy-octosdi"
 				(path "/cb0cdcc9-6b9b-4b74-8146-9043de7999b1/731e7cbd-3c26-4319-8367-0b2702130274"
-					(reference "R67")
+					(reference "R80")
 					(unit 1)
 				)
@@
 		(dnp no)
 		(fields_autoplaced yes)
-		(property "Reference" "#PWR0117"
+		(property "Reference" "#PWR0124"
 			(at 102.87 123.19 0)
 			(hide yes)
@@
 			(project "syzygy-octosdi"
 				(path "/cb0cdcc9-6b9b-4b74-8146-9043de7999b1/731e7cbd-3c26-4319-8367-0b2702130274"
-					(reference "#PWR0117")
+					(reference "#PWR0124")
 					(unit 1)
 				)
@@
 		(dnp no)
 		(fields_autoplaced yes)
-		(property "Reference" "#PWR0118"
+		(property "Reference" "#PWR0125"
 			(at 102.87 135.89 0)
 			(hide yes)
@@
 			(project "syzygy-octosdi"
 				(path "/cb0cdcc9-6b9b-4b74-8146-9043de7999b1/731e7cbd-3c26-4319-8367-0b2702130274"
-					(reference "#PWR0118")
+					(reference "#PWR0125")
 					(unit 1)
 				)
@@
 		(dnp no)
 		(fields_autoplaced yes)
-		(property "Reference" "#PWR0112"
+		(property "Reference" "#PWR0119"
 			(at 58.42 146.05 0)
 			(hide yes)
@@
 			(project "syzygy-octosdi"
 				(path "/cb0cdcc9-6b9b-4b74-8146-9043de7999b1/731e7cbd-3c26-4319-8367-0b2702130274"
-					(reference "#PWR0112")
+					(reference "#PWR0119")
 					(unit 1)
 				)
@@
 		(dnp no)
 		(fields_autoplaced yes)
-		(property "Reference" "#PWR0115"
+		(property "Reference" "#PWR0122"
 			(at 97.79 43.18 0)
 			(hide yes)
@@
 			(project "syzygy-octosdi"
 				(path "/cb0cdcc9-6b9b-4b74-8146-9043de7999b1/731e7cbd-3c26-4319-8367-0b2702130274"
-					(reference "#PWR0115")
+					(reference "#PWR0122")
 					(unit 1)
 				)
@@
 		(in_pos_files yes)
 		(dnp no)
-		(property "Reference" "R63"
+		(property "Reference" "R77"
 			(at 60.96 121.9199 0)
 			(show_name no)
@@
 			(project "syzygy-octosdi"
 				(path "/cb0cdcc9-6b9b-4b74-8146-9043de7999b1/731e7cbd-3c26-4319-8367-0b2702130274"
-					(reference "R63")
+					(reference "R77")
 					(unit 1)
 				)
@@
 		(in_pos_files yes)
 		(dnp no)
-		(property "Reference" "R70"
+		(property "Reference" "R82"
 			(at 185.42 119.3799 0)
 			(show_name no)
@@
 			(project "syzygy-octosdi"
 				(path "/cb0cdcc9-6b9b-4b74-8146-9043de7999b1/731e7cbd-3c26-4319-8367-0b2702130274"
-					(reference "R70")
+					(reference "R82")
 					(unit 1)
 				)
@@
 		(in_pos_files yes)
 		(dnp no)
-		(property "Reference" "C66"
+		(property "Reference" "C82"
 			(at 69.85 50.8062 0)
 			(show_name no)
@@
 			(project "syzygy-octosdi"
 				(path "/cb0cdcc9-6b9b-4b74-8146-9043de7999b1/731e7cbd-3c26-4319-8367-0b2702130274"
-					(reference "C66")
+					(reference "C82")
 					(unit 1)
 				)
@@
 		(in_pos_files yes)
 		(dnp no)
-		(property "Reference" "R65"
+		(property "Reference" "R79"
 			(at 110.49 166.3699 0)
 			(show_name no)
@@
 			(project "syzygy-octosdi"
 				(path "/cb0cdcc9-6b9b-4b74-8146-9043de7999b1/731e7cbd-3c26-4319-8367-0b2702130274"
-					(reference "R65")
+					(reference "R79")
 					(unit 1)
 				)
@@
 		(dnp yes)
 		(fields_autoplaced yes)
-		(property "Reference" "J1"
+		(property "Reference" "J9"
 			(at 57.15 161.29 0)
 			(show_name no)
@@
 			(project "syzygy-octosdi"
 				(path "/cb0cdcc9-6b9b-4b74-8146-9043de7999b1/731e7cbd-3c26-4319-8367-0b2702130274"
-					(reference "J1")
+					(reference "J9")
 					(unit 1)
 				)
@@
 		(dnp no)
 		(fields_autoplaced yes)
-		(property "Reference" "#PWR0110"
+		(property "Reference" "#PWR0117"
 			(at 43.18 168.91 0)
 			(hide yes)
@@
 			(project "syzygy-octosdi"
 				(path "/cb0cdcc9-6b9b-4b74-8146-9043de7999b1/731e7cbd-3c26-4319-8367-0b2702130274"
-					(reference "#PWR0110")
+					(reference "#PWR0117")
 					(unit 1)
 				)
@@
 		(in_pos_files yes)
 		(dnp no)
-		(property "Reference" "R66"
+		(property "Reference" "R81"
 			(at 160.02 125.7299 0)
 			(show_name no)
@@
 			(project "syzygy-octosdi"
 				(path "/cb0cdcc9-6b9b-4b74-8146-9043de7999b1/731e7cbd-3c26-4319-8367-0b2702130274"
-					(reference "R66")
+					(reference "R81")
 					(unit 1)
 				)
@@
 		(dnp no)
 		(fields_autoplaced yes)
-		(property "Reference" "#PWR0113"
+		(property "Reference" "#PWR0120"
 			(at 72.39 60.96 0)
 			(hide yes)
@@
 			(project "syzygy-octosdi"
 				(path "/cb0cdcc9-6b9b-4b74-8146-9043de7999b1/731e7cbd-3c26-4319-8367-0b2702130274"
-					(reference "#PWR0113")
+					(reference "#PWR0120")
 					(unit 1)
 				)
@@
 		(dnp no)
 		(fields_autoplaced yes)
-		(property "Reference" "#PWR0114"
+		(property "Reference" "#PWR0121"
 			(at 76.2 146.05 0)
 			(hide yes)
@@
 			(project "syzygy-octosdi"
 				(path "/cb0cdcc9-6b9b-4b74-8146-9043de7999b1/731e7cbd-3c26-4319-8367-0b2702130274"
-					(reference "#PWR0114")
+					(reference "#PWR0121")
 					(unit 1)
 				)
@@
 		(dnp no)
 		(fields_autoplaced yes)
-		(property "Reference" "#PWR0111"
+		(property "Reference" "#PWR0118"
 			(at 43.18 179.07 0)
 			(hide yes)
@@
 			(project "syzygy-octosdi"
 				(path "/cb0cdcc9-6b9b-4b74-8146-9043de7999b1/731e7cbd-3c26-4319-8367-0b2702130274"
-					(reference "#PWR0111")
+					(reference "#PWR0118")
 					(unit 1)
 				)
@@
 		(dnp no)
 		(fields_autoplaced yes)
-		(property "Reference" "#PWR0128"
+		(property "Reference" "#PWR0129"
 			(at 182.88 143.51 0)
 			(hide yes)
@@
 			(project "syzygy-octosdi"
 				(path "/cb0cdcc9-6b9b-4b74-8146-9043de7999b1/731e7cbd-3c26-4319-8367-0b2702130274"
-					(reference "#PWR0128")
+					(reference "#PWR0129")
 					(unit 1)
 				)
@@
 		(dnp no)
 		(fields_autoplaced yes)
-		(property "Reference" "#PWR0116"
+		(property "Reference" "#PWR0123"
 			(at 97.79 95.25 0)
 			(hide yes)
@@
 			(project "syzygy-octosdi"
 				(path "/cb0cdcc9-6b9b-4b74-8146-9043de7999b1/731e7cbd-3c26-4319-8367-0b2702130274"
-					(reference "#PWR0116")
+					(reference "#PWR0123")
 					(unit 1)
 				)
@@
 		(dnp no)
 		(fields_autoplaced yes)
-		(property "Reference" "#PWR0119"
+		(property "Reference" "#PWR0126"
 			(at 107.95 166.37 0)
 			(hide yes)
@@
 			(project "syzygy-octosdi"
 				(path "/cb0cdcc9-6b9b-4b74-8146-9043de7999b1/731e7cbd-3c26-4319-8367-0b2702130274"
-					(reference "#PWR0119")
+					(reference "#PWR0126")
 					(unit 1)
 				)
@@
 		(dnp no)
 		(fields_autoplaced yes)
-		(property "Reference" "C67"
+		(property "Reference" "C83"
 			(at 105.41 123.1962 0)
 			(show_name no)
@@
 			(project "syzygy-octosdi"
 				(path "/cb0cdcc9-6b9b-4b74-8146-9043de7999b1/731e7cbd-3c26-4319-8367-0b2702130274"
-					(reference "C67")
+					(reference "C83")
 					(unit 1)
 				)
@@
 		(in_pos_files yes)
 		(dnp no)
-		(property "Reference" "R64"
+		(property "Reference" "R78"
 			(at 78.74 121.9199 0)
 			(show_name no)
@@
 			(project "syzygy-octosdi"
 				(path "/cb0cdcc9-6b9b-4b74-8146-9043de7999b1/731e7cbd-3c26-4319-8367-0b2702130274"
-					(reference "R64")
-					(unit 1)
-				)
+					(reference "R78")
+					(unit 1)
+				)

Commit message: split gpio expanders by inputs/outputs instead of quads
Parts:
- C82, C83, C84, D10, D11, D9, R77, R78, R79, R80, R81, R82: KiLib_Generator (none) -> SMD_2terminal_chip_molded
- J9: KiLib_Generator (none) -> connector/pin_header_socket
- U11: KiLib_Generator (none) -> package/no_lead
Changed lines of the file:
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@@
+			)
+		)
+		(property "KiLib_Generator" "package/no_lead"
+			(at 97.79 66.04 0)
+			(hide yes)
+			(show_name no)
+			(do_not_autoplace no)
+			(effects
+				(font
+					(size 1.27 1.27)
+				)
 			)
 		)
@@
 		)
 		(property "Sim.Pins" "1=K 2=A"
+			(at 182.88 130.81 0)
+			(hide yes)
+			(show_name no)
+			(do_not_autoplace no)
+			(effects
+				(font
+					(size 1.27 1.27)
+				)
+			)
+		)
+		(property "KiLib_Generator" "SMD_2terminal_chip_molded"
 			(at 182.88 130.81 0)
 			(hide yes)
@@
 			)
 		)
+		(property "KiLib_Generator" "SMD_2terminal_chip_molded"
+			(at 111.76 124.46 0)
+			(hide yes)
+			(show_name no)
+			(do_not_autoplace no)
+			(effects
+				(font
+					(size 1.27 1.27)
+				)
+			)
+		)
 		(pin "1"
 		)
@@
 		)
 		(property "Description" "Resistor"
+			(at 138.43 129.54 0)
+			(hide yes)
+			(show_name no)
+			(do_not_autoplace no)
+			(effects
+				(font
+					(size 1.27 1.27)
+				)
+			)
+		)
+		(property "KiLib_Generator" "SMD_2terminal_chip_molded"
 			(at 138.43 129.54 0)
 			(hide yes)
@@
 			)
 		)
+		(property "KiLib_Generator" "SMD_2terminal_chip_molded"
+			(at 76.2 133.35 0)
+			(hide yes)
+			(show_name no)
+			(do_not_autoplace no)
+			(effects
+				(font
+					(size 1.27 1.27)
+				)
+			)
+		)
 		(pin "1"
 		)
@@
 			)
 		)
+		(property "KiLib_Generator" "SMD_2terminal_chip_molded"
+			(at 58.42 123.19 0)
+			(hide yes)
+			(show_name no)
+			(do_not_autoplace no)
+			(effects
+				(font
+					(size 1.27 1.27)
+				)
+			)
+		)
 		(pin "1"
 		)
@@
 		)
 		(property "Description" "Resistor"
+			(at 182.88 120.65 0)
+			(hide yes)
+			(show_name no)
+			(do_not_autoplace no)
+			(effects
+				(font
+					(size 1.27 1.27)
+				)
+			)
+		)
+		(property "KiLib_Generator" "SMD_2terminal_chip_molded"
 			(at 182.88 120.65 0)
 			(hide yes)
@@
 			)
 		)
+		(property "KiLib_Generator" "SMD_2terminal_chip_molded"
+			(at 72.39 52.07 0)
+			(hide yes)
+			(show_name no)
+			(do_not_autoplace no)
+			(effects
+				(font
+					(size 1.27 1.27)
+				)
+			)
+		)
 		(pin "2"
 		)
@@
 		)
 		(property "Description" "Resistor"
+			(at 107.95 167.64 0)
+			(hide yes)
+			(show_name no)
+			(do_not_autoplace no)
+			(effects
+				(font
+					(size 1.27 1.27)
+				)
+			)
+		)
+		(property "KiLib_Generator" "SMD_2terminal_chip_molded"
 			(at 107.95 167.64 0)
 			(hide yes)
@@
 			)
 		)
+		(property "KiLib_Generator" "connector/pin_header_socket"
+			(at 55.88 170.18 0)
+			(hide yes)
+			(show_name no)
+			(do_not_autoplace no)
+			(effects
+				(font
+					(size 1.27 1.27)
+				)
+			)
+		)
 		(pin "1"
 		)
@@
 			)
 		)
+		(property "KiLib_Generator" "SMD_2terminal_chip_molded"
+			(at 162.56 127 0)
+			(hide yes)
+			(show_name no)
+			(do_not_autoplace no)
+			(effects
+				(font
+					(size 1.27 1.27)
+				)
+			)
+		)
 		(pin "1"
 		)
@@
 			)
 		)
+		(property "KiLib_Generator" "SMD_2terminal_chip_molded"
+			(at 58.42 133.35 0)
+			(hide yes)
+			(show_name no)
+			(do_not_autoplace no)
+			(effects
+				(font
+					(size 1.27 1.27)
+				)
+			)
+		)
 		(pin "1"
 		)
@@
 			)
 		)
+		(property "KiLib_Generator" "SMD_2terminal_chip_molded"
+			(at 102.87 124.46 0)
+			(hide yes)
+			(show_name no)
+			(do_not_autoplace no)
+			(effects
+				(font
+					(size 1.27 1.27)
+				)
+			)
+		)
 		(pin "1"
 		)
@@
 			(at 76.2 123.19 0)
 			(hide yes)
+			(show_name no)
+			(do_not_autoplace no)
+			(effects
+				(font
+					(size 1.27 1.27)
+				)
+			)
+		)
+		(property "KiLib_Generator" "SMD_2terminal_chip_molded"
+			(at 76.2 123.19 0)
+			(hide yes)

Commit message: route the smartvio mcu and the gpio expanders
Changed lines of the file:
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@@
 		)
 	)
-	(text_box "Programming Header"
+	(text_box "Programming Header\nData lines to PCB edge"
 		(exclude_from_sim no)
 		(at 35.56 153.67 0)

Commit message: fixes following review and more mounting holes
Parts:
- U11: footprint Package_DFN_QFN:QFN-28_4x4mm_P0.5mm -> JLCImport:UFQFPN-28_STM
Changed lines of the file:
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@@
 			)
 		)
-		(property "Footprint" "Package_DFN_QFN:QFN-28_4x4mm_P0.5mm"
+		(property "Footprint" "JLCImport:UFQFPN-28_STM"
 			(at 82.55 86.36 0)
 			(hide yes)

Commit message: add power led and test points
Parts:
- renumbered C82 to C84, C83 to C85, C84 to C86, D9 to D10, D10 to D11, D11 to D12, R77 to R78, R78 to R79, R79 to R80, R80 to R81, R81 to R82, R82 to R83, TP1 to TP13, TP2 to TP14
Changed lines of the file:
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@@
 		(in_pos_files yes)
 		(dnp no)
-		(property "Reference" "TP1"
+		(property "Reference" "TP13"
 			(at 52.07 57.6579 0)
 			(show_name no)
@@
 			(project "syzygy-octosdi"
 				(path "/cb0cdcc9-6b9b-4b74-8146-9043de7999b1/731e7cbd-3c26-4319-8367-0b2702130274"
-					(reference "TP1")
+					(reference "TP13")
 					(unit 1)
 				)
@@
 		(dnp no)
 		(fields_autoplaced yes)
-		(property "Reference" "#PWR0128"
+		(property "Reference" "#PWR0134"
 			(at 162.56 138.43 0)
 			(hide yes)
@@
 			(project "syzygy-octosdi"
 				(path "/cb0cdcc9-6b9b-4b74-8146-9043de7999b1/731e7cbd-3c26-4319-8367-0b2702130274"
-					(reference "#PWR0128")
+					(reference "#PWR0134")
 					(unit 1)
 				)
@@
 		(in_pos_files yes)
 		(dnp no)
-		(property "Reference" "D11"
+		(property "Reference" "D12"
 			(at 186.69 131.1274 90)
 			(show_name no)
@@
 			(project "syzygy-octosdi"
 				(path "/cb0cdcc9-6b9b-4b74-8146-9043de7999b1/731e7cbd-3c26-4319-8367-0b2702130274"
-					(reference "D11")
+					(reference "D12")
 					(unit 1)
 				)
@@
 		(dnp no)
 		(fields_autoplaced yes)
-		(property "Reference" "C84"
+		(property "Reference" "C86"
 			(at 114.3 123.1962 0)
 			(show_name no)
@@
 			(project "syzygy-octosdi"
 				(path "/cb0cdcc9-6b9b-4b74-8146-9043de7999b1/731e7cbd-3c26-4319-8367-0b2702130274"
-					(reference "C84")
+					(reference "C86")
 					(unit 1)
 				)
@@
 		(in_pos_files yes)
 		(dnp no)
-		(property "Reference" "R80"
+		(property "Reference" "R81"
 			(at 135.89 128.2699 0)
 			(show_name no)
@@
 			(project "syzygy-octosdi"
 				(path "/cb0cdcc9-6b9b-4b74-8146-9043de7999b1/731e7cbd-3c26-4319-8367-0b2702130274"
-					(reference "R80")
+					(reference "R81")
 					(unit 1)
 				)
@@
 		(dnp no)
 		(fields_autoplaced yes)
-		(property "Reference" "#PWR0124"
+		(property "Reference" "#PWR0130"
 			(at 102.87 123.19 0)
 			(hide yes)
@@
 			(project "syzygy-octosdi"
 				(path "/cb0cdcc9-6b9b-4b74-8146-9043de7999b1/731e7cbd-3c26-4319-8367-0b2702130274"
-					(reference "#PWR0124")
+					(reference "#PWR0130")
 					(unit 1)
 				)
@@
 		(dnp no)
 		(fields_autoplaced yes)
-		(property "Reference" "#PWR0125"
+		(property "Reference" "#PWR0131"
 			(at 102.87 135.89 0)
 			(hide yes)
@@
 			(project "syzygy-octosdi"
 				(path "/cb0cdcc9-6b9b-4b74-8146-9043de7999b1/731e7cbd-3c26-4319-8367-0b2702130274"
-					(reference "#PWR0125")
+					(reference "#PWR0131")
 					(unit 1)
 				)
@@
 		(dnp no)
 		(fields_autoplaced yes)
-		(property "Reference" "#PWR0119"
+		(property "Reference" "#PWR0125"
 			(at 58.42 146.05 0)
 			(hide yes)
@@
 			(project "syzygy-octosdi"
 				(path "/cb0cdcc9-6b9b-4b74-8146-9043de7999b1/731e7cbd-3c26-4319-8367-0b2702130274"
-					(reference "#PWR0119")
+					(reference "#PWR0125")
 					(unit 1)
 				)
@@
 		(dnp no)
 		(fields_autoplaced yes)
-		(property "Reference" "#PWR0122"
+		(property "Reference" "#PWR0128"
 			(at 97.79 43.18 0)
 			(hide yes)
@@
 			(project "syzygy-octosdi"
 				(path "/cb0cdcc9-6b9b-4b74-8146-9043de7999b1/731e7cbd-3c26-4319-8367-0b2702130274"
-					(reference "#PWR0122")
+					(reference "#PWR0128")
 					(unit 1)
 				)
@@
 		(in_pos_files yes)
 		(dnp no)
-		(property "Reference" "D10"
+		(property "Reference" "D11"
 			(at 80.01 133.6674 90)
 			(show_name no)
@@
 			(project "syzygy-octosdi"
 				(path "/cb0cdcc9-6b9b-4b74-8146-9043de7999b1/731e7cbd-3c26-4319-8367-0b2702130274"
-					(reference "D10")
+					(reference "D11")
 					(unit 1)
 				)
@@
 		(in_pos_files yes)
 		(dnp no)
-		(property "Reference" "R77"
+		(property "Reference" "R78"
 			(at 60.96 121.9199 0)
 			(show_name no)
@@
 			(project "syzygy-octosdi"
 				(path "/cb0cdcc9-6b9b-4b74-8146-9043de7999b1/731e7cbd-3c26-4319-8367-0b2702130274"
-					(reference "R77")
+					(reference "R78")
 					(unit 1)
 				)
@@
 		(in_pos_files yes)
 		(dnp no)
-		(property "Reference" "R82"
+		(property "Reference" "R83"
 			(at 185.42 119.3799 0)
 			(show_name no)
@@
 			(project "syzygy-octosdi"
 				(path "/cb0cdcc9-6b9b-4b74-8146-9043de7999b1/731e7cbd-3c26-4319-8367-0b2702130274"
-					(reference "R82")
+					(reference "R83")
 					(unit 1)
 				)
@@
 		(in_pos_files yes)
 		(dnp no)
-		(property "Reference" "C82"
+		(property "Reference" "C84"
 			(at 69.85 50.8062 0)
 			(show_name no)
@@
 			(project "syzygy-octosdi"
 				(path "/cb0cdcc9-6b9b-4b74-8146-9043de7999b1/731e7cbd-3c26-4319-8367-0b2702130274"
-					(reference "C82")
+					(reference "C84")
 					(unit 1)
 				)
@@
 		(in_pos_files yes)
 		(dnp no)
-		(property "Reference" "R79"
+		(property "Reference" "R80"
 			(at 110.49 166.3699 0)
 			(show_name no)
@@
 			(project "syzygy-octosdi"
 				(path "/cb0cdcc9-6b9b-4b74-8146-9043de7999b1/731e7cbd-3c26-4319-8367-0b2702130274"
-					(reference "R79")
+					(reference "R80")
 					(unit 1)
 				)
@@
 		(dnp no)
 		(fields_autoplaced yes)
-		(property "Reference" "#PWR0117"
+		(property "Reference" "#PWR0123"
 			(at 43.18 168.91 0)
 			(hide yes)
@@
 			(project "syzygy-octosdi"
 				(path "/cb0cdcc9-6b9b-4b74-8146-9043de7999b1/731e7cbd-3c26-4319-8367-0b2702130274"
-					(reference "#PWR0117")
+					(reference "#PWR0123")
 					(unit 1)
 				)
@@
 		(in_pos_files yes)
 		(dnp no)
-		(property "Reference" "R81"
+		(property "Reference" "R82"
 			(at 160.02 125.7299 0)
 			(show_name no)
@@
 			(project "syzygy-octosdi"
 				(path "/cb0cdcc9-6b9b-4b74-8146-9043de7999b1/731e7cbd-3c26-4319-8367-0b2702130274"
-					(reference "R81")
+					(reference "R82")
 					(unit 1)
 				)
@@
 		(dnp no)
 		(fields_autoplaced yes)
-		(property "Reference" "#PWR0120"
+		(property "Reference" "#PWR0126"
 			(at 72.39 60.96 0)
 			(hide yes)
@@
 			(project "syzygy-octosdi"
 				(path "/cb0cdcc9-6b9b-4b74-8146-9043de7999b1/731e7cbd-3c26-4319-8367-0b2702130274"
-					(reference "#PWR0120")
+					(reference "#PWR0126")
 					(unit 1)
 				)
@@
 		(dnp no)
 		(fields_autoplaced yes)
-		(property "Reference" "TP2"
+		(property "Reference" "TP14"
 			(at 60.96 57.6579 0)
 			(show_name no)
@@
 			(project "syzygy-octosdi"
 				(path "/cb0cdcc9-6b9b-4b74-8146-9043de7999b1/731e7cbd-3c26-4319-8367-0b2702130274"
-					(reference "TP2")
+					(reference "TP14")
 					(unit 1)
 				)
@@
 		(dnp no)
 		(fields_autoplaced yes)
-		(property "Reference" "#PWR0121"
+		(property "Reference" "#PWR0127"
 			(at 76.2 146.05 0)
 			(hide yes)
@@
 			(project "syzygy-octosdi"
 				(path "/cb0cdcc9-6b9b-4b74-8146-9043de7999b1/731e7cbd-3c26-4319-8367-0b2702130274"
-					(reference "#PWR0121")
+					(reference "#PWR0127")
 					(unit 1)
 				)
@@
 		(dnp no)
 		(fields_autoplaced yes)
-		(property "Reference" "#PWR0118"
+		(property "Reference" "#PWR0124"
 			(at 43.18 179.07 0)
 			(hide yes)
@@
 			(project "syzygy-octosdi"
 				(path "/cb0cdcc9-6b9b-4b74-8146-9043de7999b1/731e7cbd-3c26-4319-8367-0b2702130274"
-					(reference "#PWR0118")
+					(reference "#PWR0124")
 					(unit 1)
 				)
@@
 		(dnp no)
 		(fields_autoplaced yes)
-		(property "Reference" "#PWR0129"
+		(property "Reference" "#PWR0135"
 			(at 182.88 143.51 0)
 			(hide yes)
@@
 			(project "syzygy-octosdi"
 				(path "/cb0cdcc9-6b9b-4b74-8146-9043de7999b1/731e7cbd-3c26-4319-8367-0b2702130274"
-					(reference "#PWR0129")
+					(reference "#PWR0135")
 					(unit 1)
 				)
@@
 		(dnp no)
 		(fields_autoplaced yes)
-		(property "Reference" "#PWR0127"
+		(property "Reference" "#PWR0133"
 			(at 138.43 128.27 0)
 			(hide yes)
@@
 			(project "syzygy-octosdi"
 				(path "/cb0cdcc9-6b9b-4b74-8146-9043de7999b1/731e7cbd-3c26-4319-8367-0b2702130274"
-					(reference "#PWR0127")
+					(reference "#PWR0133")
 					(unit 1)
 				)
@@
 		(dnp no)
 		(fields_autoplaced yes)
-		(property "Reference" "#PWR0123"
+		(property "Reference" "#PWR0129"
 			(at 97.79 95.25 0)
 			(hide yes)
@@
 			(project "syzygy-octosdi"
 				(path "/cb0cdcc9-6b9b-4b74-8146-9043de7999b1/731e7cbd-3c26-4319-8367-0b2702130274"
-					(reference "#PWR0123")
+					(reference "#PWR0129")
 					(unit 1)
 				)
@@
 		(dnp no)
 		(fields_autoplaced yes)
-		(property "Reference" "#PWR0126"
+		(property "Reference" "#PWR0132"
 			(at 107.95 166.37 0)
 			(hide yes)
@@
 			(project "syzygy-octosdi"
 				(path "/cb0cdcc9-6b9b-4b74-8146-9043de7999b1/731e7cbd-3c26-4319-8367-0b2702130274"
-					(reference "#PWR0126")
+					(reference "#PWR0132")
 					(unit 1)
 				)
@@
 		(in_pos_files yes)
 		(dnp no)
-		(property "Reference" "D9"
+		(property "Reference" "D10"
 			(at 62.23 133.6674 90)
 			(show_name no)
@@
 			(project "syzygy-octosdi"
 				(path "/cb0cdcc9-6b9b-4b74-8146-9043de7999b1/731e7cbd-3c26-4319-8367-0b2702130274"
-					(reference "D9")
+					(reference "D10")
 					(unit 1)
 				)
@@
 		(dnp no)
 		(fields_autoplaced yes)
-		(property "Reference" "C83"
+		(property "Reference" "C85"
 			(at 105.41 123.1962 0)
 			(show_name no)
@@
 			(project "syzygy-octosdi"
 				(path "/cb0cdcc9-6b9b-4b74-8146-9043de7999b1/731e7cbd-3c26-4319-8367-0b2702130274"
-					(reference "C83")
+					(reference "C85")
 					(unit 1)
 				)
@@
 		(in_pos_files yes)
 		(dnp no)
-		(property "Reference" "R78"
+		(property "Reference" "R79"
 			(at 78.74 121.9199 0)
 			(show_name no)
@@
 			(project "syzygy-octosdi"
 				(path "/cb0cdcc9-6b9b-4b74-8146-9043de7999b1/731e7cbd-3c26-4319-8367-0b2702130274"
-					(reference "R78")
-					(unit 1)
-				)
+					(reference "R79")
+					(unit 1)
+				)

Commit message: check against jlcpcb capabilities
Parts:
- J9: now fitted; now left out of the parts list
- TP13, TP14: now left out of the parts list
Changed lines of the file:
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@@
 		(body_style 1)
 		(exclude_from_sim no)
-		(in_bom yes)
+		(in_bom no)
 		(on_board yes)
 		(in_pos_files yes)
@@
 		(body_style 1)
 		(exclude_from_sim no)
-		(in_bom yes)
-		(on_board yes)
-		(in_pos_files yes)
-		(dnp yes)
+		(in_bom no)
+		(on_board yes)
+		(in_pos_files yes)
+		(dnp no)
 		(fields_autoplaced yes)
 		(property "Reference" "J9"
@@
 		(body_style 1)
 		(exclude_from_sim no)
-		(in_bom yes)
-		(on_board yes)
-		(in_pos_files yes)
+		(in_bom no)
+		(on_board yes)
+		(in_pos_files yes)
