File: smartvio.kicad_sch (KiCad schematic)
At the start: 16 parts, among them J9 Conn_02x03_Odd_Even, U11 STM32G031G8Ux

Commit message: specify skus for parts
Parts:
- C85, C87: LCSC (none) -> C282519
- C86: LCSC (none) -> C69335
- R78, R79, R83: LCSC (none) -> C2907034
- R80, R81, R82: LCSC (none) -> C25804
- U11: LCSC (none) -> C432211
Changed lines of the file:
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@@
+			)
+		)
+		(property "LCSC" "C432211"
+			(at 97.79 66.04 0)
+			(hide yes)
+			(show_name no)
+			(do_not_autoplace no)
+			(effects
+				(font
+					(size 1.27 1.27)
+				)
 			)
 		)
@@
 			)
 		)
+		(property "LCSC" "C282519"
+			(at 111.76 124.46 0)
+			(hide yes)
+			(show_name no)
+			(do_not_autoplace no)
+			(effects
+				(font
+					(size 1.27 1.27)
+				)
+			)
+		)
 		(pin "1"
 		)
@@
 		)
 		(property "KiLib_Generator" "SMD_2terminal_chip_molded"
+			(at 138.43 129.54 0)
+			(hide yes)
+			(show_name no)
+			(do_not_autoplace no)
+			(effects
+				(font
+					(size 1.27 1.27)
+				)
+			)
+		)
+		(property "LCSC" "C25804"
 			(at 138.43 129.54 0)
 			(hide yes)
@@
 			)
 		)
+		(property "LCSC" "C2907034"
+			(at 58.42 123.19 0)
+			(hide yes)
+			(show_name no)
+			(do_not_autoplace no)
+			(effects
+				(font
+					(size 1.27 1.27)
+				)
+			)
+		)
 		(pin "1"
 		)
@@
 		)
 		(property "KiLib_Generator" "SMD_2terminal_chip_molded"
+			(at 182.88 120.65 0)
+			(hide yes)
+			(show_name no)
+			(do_not_autoplace no)
+			(effects
+				(font
+					(size 1.27 1.27)
+				)
+			)
+		)
+		(property "LCSC" "C2907034"
 			(at 182.88 120.65 0)
 			(hide yes)
@@
 			)
 		)
+		(property "LCSC" "C282519"
+			(at 72.39 52.07 0)
+			(hide yes)
+			(show_name no)
+			(do_not_autoplace no)
+			(effects
+				(font
+					(size 1.27 1.27)
+				)
+			)
+		)
 		(pin "2"
 		)
@@
 		)
 		(property "KiLib_Generator" "SMD_2terminal_chip_molded"
+			(at 107.95 167.64 0)
+			(hide yes)
+			(show_name no)
+			(do_not_autoplace no)
+			(effects
+				(font
+					(size 1.27 1.27)
+				)
+			)
+		)
+		(property "LCSC" "C25804"
 			(at 107.95 167.64 0)
 			(hide yes)
@@
 			)
 		)
+		(property "LCSC" "C25804"
+			(at 162.56 127 0)
+			(hide yes)
+			(show_name no)
+			(do_not_autoplace no)
+			(effects
+				(font
+					(size 1.27 1.27)
+				)
+			)
+		)
 		(pin "1"
 		)
@@
 			)
 		)
+		(property "LCSC" "C69335"
+			(at 102.87 124.46 0)
+			(hide yes)
+			(show_name no)
+			(do_not_autoplace no)
+			(effects
+				(font
+					(size 1.27 1.27)
+				)
+			)
+		)
 		(pin "1"
 		)
@@
 			(at 76.2 123.19 0)
 			(hide yes)
+			(show_name no)
+			(do_not_autoplace no)
+			(effects
+				(font
+					(size 1.27 1.27)
+				)
+			)
+		)
+		(property "LCSC" "C2907034"
+			(at 76.2 123.19 0)
+			(hide yes)

Commit message: specify led colours
Parts:
- D10, D11: value LED -> LED Green
- D12: value LED -> LED Orange
Other:
- moved on the sheet: D10, D11, R78, R79
Changed lines of the file:
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@@
 		(exclude_from_sim no)
 		(at 129.54 106.68 0)
-		(size 64.77 43.18)
+		(size 69.85 43.18)
 		(margins 0.9525 0.9525 0.9525 0.9525)
 		(stroke
@@
 		(exclude_from_sim no)
 		(at 35.56 106.68 0)
-		(size 52.07 43.18)
+		(size 54.61 43.18)
 		(margins 0.9525 0.9525 0.9525 0.9525)
 		(stroke
@@
 	(wire
 		(pts
-			(xy 76.2 116.84) (xy 76.2 119.38)
+			(xy 73.66 116.84) (xy 73.66 119.38)
 		)
 		(stroke
@@
 	(wire
 		(pts
-			(xy 44.45 116.84) (xy 58.42 116.84)
+			(xy 41.91 116.84) (xy 55.88 116.84)
 		)
 		(stroke
@@
 	(wire
 		(pts
-			(xy 76.2 137.16) (xy 76.2 139.7)
+			(xy 73.66 137.16) (xy 73.66 139.7)
 		)
 		(stroke
@@
 	(wire
 		(pts
-			(xy 62.23 116.84) (xy 76.2 116.84)
+			(xy 59.69 116.84) (xy 73.66 116.84)
 		)
 		(stroke
@@
 	(wire
 		(pts
-			(xy 58.42 137.16) (xy 58.42 139.7)
+			(xy 55.88 137.16) (xy 55.88 139.7)
 		)
 		(stroke
@@
 	(wire
 		(pts
-			(xy 58.42 116.84) (xy 58.42 119.38)
+			(xy 55.88 116.84) (xy 55.88 119.38)
 		)
 		(stroke
@@
 	(wire
 		(pts
-			(xy 76.2 127) (xy 76.2 129.54)
+			(xy 73.66 127) (xy 73.66 129.54)
 		)
 		(stroke
@@
 	(wire
 		(pts
-			(xy 58.42 127) (xy 58.42 129.54)
+			(xy 55.88 127) (xy 55.88 129.54)
 		)
 		(stroke
@@
 	)
 	(label "USER_LED_0"
-		(at 62.23 116.84 0)
+		(at 59.69 116.84 0)
 		(effects
 			(font
@@
 	)
 	(label "USER_LED_1"
-		(at 44.45 116.84 0)
+		(at 41.91 116.84 0)
 		(effects
 			(font
@@
 			)
 		)
-		(property "Value" "LED"
+		(property "Value" "LED Orange"
 			(at 186.69 133.6674 90)
 			(show_name no)
@@
 	(symbol
 		(lib_id "power:GND")
-		(at 58.42 139.7 0)
+		(at 55.88 139.7 0)
 		(unit 1)
 		(body_style 1)
@@
 		(fields_autoplaced yes)
 		(property "Reference" "#PWR0127"
-			(at 58.42 146.05 0)
+			(at 55.88 146.05 0)
 			(hide yes)
 			(show_name no)
@@
 		)
 		(property "Value" "GND"
-			(at 58.42 144.78 0)
+			(at 55.88 144.78 0)
 			(show_name no)
 			(do_not_autoplace no)
@@
 		)
 		(property "Footprint" ""
-			(at 58.42 139.7 0)
+			(at 55.88 139.7 0)
 			(hide yes)
 			(show_name no)
@@
 		)
 		(property "Datasheet" ""
-			(at 58.42 139.7 0)
+			(at 55.88 139.7 0)
 			(hide yes)
 			(show_name no)
@@
 		)
 		(property "Description" "Power symbol creates a global label with name \"GND\" , ground"
-			(at 58.42 139.7 0)
+			(at 55.88 139.7 0)
 			(hide yes)
 			(show_name no)
@@
 	(symbol
 		(lib_id "Device:LED")
-		(at 76.2 133.35 90)
+		(at 73.66 133.35 90)
 		(unit 1)
 		(body_style 1)
@@
 		(dnp no)
 		(property "Reference" "D11"
-			(at 80.01 133.6674 90)
+			(at 77.47 133.6674 90)
 			(show_name no)
 			(do_not_autoplace no)
@@
 			)
 		)
-		(property "Value" "LED"
-			(at 80.01 136.2074 90)
+		(property "Value" "LED Green"
+			(at 77.47 136.2074 90)
 			(show_name no)
 			(do_not_autoplace no)
@@
 		)
 		(property "Footprint" "LED_SMD:LED_0603_1608Metric"
-			(at 76.2 133.35 0)
+			(at 73.66 133.35 0)
 			(hide yes)
 			(show_name no)
@@
 		)
 		(property "Datasheet" ""
-			(at 76.2 133.35 0)
+			(at 73.66 133.35 0)
 			(hide yes)
 			(show_name no)
@@
 		)
 		(property "Description" "Light emitting diode"
-			(at 76.2 133.35 0)
+			(at 73.66 133.35 0)
 			(hide yes)
 			(show_name no)
@@
 		)
 		(property "Sim.Pins" "1=K 2=A"
-			(at 76.2 133.35 0)
+			(at 73.66 133.35 0)
 			(hide yes)
 			(show_name no)
@@
 		)
 		(property "KiLib_Generator" "SMD_2terminal_chip_molded"
-			(at 76.2 133.35 0)
+			(at 73.66 133.35 0)
 			(hide yes)
 			(show_name no)
@@
 	(symbol
 		(lib_id "Device:R")
-		(at 58.42 123.19 0)
+		(at 55.88 123.19 0)
 		(unit 1)
 		(body_style 1)
@@
 		(dnp no)
 		(property "Reference" "R78"
-			(at 60.96 121.9199 0)
+			(at 58.42 121.9199 0)
 			(show_name no)
 			(do_not_autoplace no)
@@
 		)
 		(property "Value" "4k7"
-			(at 60.96 124.4599 0)
+			(at 58.42 124.4599 0)
 			(show_name no)
 			(do_not_autoplace no)
@@
 		)
 		(property "Footprint" "Resistor_SMD:R_0603_1608Metric"
-			(at 56.642 123.19 90)
+			(at 54.102 123.19 90)
 			(hide yes)
 			(show_name no)
@@
 		)
 		(property "Datasheet" ""
-			(at 58.42 123.19 0)
+			(at 55.88 123.19 0)
 			(hide yes)
 			(show_name no)
@@
 		)
 		(property "Description" "Resistor"
-			(at 58.42 123.19 0)
+			(at 55.88 123.19 0)
 			(hide yes)
 			(show_name no)
@@
 		)
 		(property "KiLib_Generator" "SMD_2terminal_chip_molded"
-			(at 58.42 123.19 0)
+			(at 55.88 123.19 0)
 			(hide yes)
 			(show_name no)
@@
 		)
 		(property "LCSC" "C2907034"
-			(at 58.42 123.19 0)
+			(at 55.88 123.19 0)
 			(hide yes)
 			(show_name no)
@@
 	(symbol
 		(lib_id "power:GND")
-		(at 76.2 139.7 0)
+		(at 73.66 139.7 0)
 		(unit 1)
 		(body_style 1)
@@
 		(fields_autoplaced yes)
 		(property "Reference" "#PWR0129"
-			(at 76.2 146.05 0)
+			(at 73.66 146.05 0)
 			(hide yes)
 			(show_name no)
@@
 		)
 		(property "Value" "GND"
-			(at 76.2 144.78 0)
+			(at 73.66 144.78 0)
 			(show_name no)
 			(do_not_autoplace no)
@@
 		)
 		(property "Footprint" ""
-			(at 76.2 139.7 0)
+			(at 73.66 139.7 0)
 			(hide yes)
 			(show_name no)
@@
 		)
 		(property "Datasheet" ""
-			(at 76.2 139.7 0)
+			(at 73.66 139.7 0)
 			(hide yes)
 			(show_name no)
@@
 		)
 		(property "Description" "Power symbol creates a global label with name \"GND\" , ground"
-			(at 76.2 139.7 0)
+			(at 73.66 139.7 0)
 			(hide yes)
 			(show_name no)
@@
 	(symbol
 		(lib_id "Device:LED")
-		(at 58.42 133.35 90)
+		(at 55.88 133.35 90)
 		(unit 1)
 		(body_style 1)
@@
 		(dnp no)
 		(property "Reference" "D10"
-			(at 62.23 133.6674 90)
+			(at 59.69 133.6674 90)
 			(show_name no)
 			(do_not_autoplace no)
@@
 			)
 		)
-		(property "Value" "LED"
-			(at 62.23 136.2074 90)
+		(property "Value" "LED Green"
+			(at 59.69 136.2074 90)
 			(show_name no)
 			(do_not_autoplace no)
@@
 		)
 		(property "Footprint" "LED_SMD:LED_0603_1608Metric"
-			(at 58.42 133.35 0)
+			(at 55.88 133.35 0)
 			(hide yes)
 			(show_name no)
@@
 		)
 		(property "Datasheet" ""
-			(at 58.42 133.35 0)
+			(at 55.88 133.35 0)
 			(hide yes)
 			(show_name no)
@@
 		)
 		(property "Description" "Light emitting diode"
-			(at 58.42 133.35 0)
+			(at 55.88 133.35 0)
 			(hide yes)
 			(show_name no)
@@
 		)
 		(property "Sim.Pins" "1=K 2=A"
-			(at 58.42 133.35 0)
+			(at 55.88 133.35 0)
 			(hide yes)
 			(show_name no)
@@
 		)
 		(property "KiLib_Generator" "SMD_2terminal_chip_molded"
-			(at 58.42 133.35 0)
+			(at 55.88 133.35 0)
 			(hide yes)
 			(show_name no)
@@
 	(symbol
 		(lib_id "Device:R")
-		(at 76.2 123.19 0)
+		(at 73.66 123.19 0)
 		(unit 1)
 		(body_style 1)
@@
 		(dnp no)
 		(property "Reference" "R79"
-			(at 78.74 121.9199 0)
+			(at 76.2 121.9199 0)
 			(show_name no)
 			(do_not_autoplace no)
@@
 		)
 		(property "Value" "4k7"
-			(at 78.74 124.4599 0)
+			(at 76.2 124.4599 0)
 			(show_name no)
 			(do_not_autoplace no)
@@
 		)
 		(property "Footprint" "Resistor_SMD:R_0603_1608Metric"
-			(at 74.422 123.19 90)
+			(at 71.882 123.19 90)
 			(hide yes)
 			(show_name no)
@@
 		)
 		(property "Datasheet" ""
-			(at 76.2 123.19 0)
+			(at 73.66 123.19 0)
 			(hide yes)
 			(show_name no)
@@
 		)
 		(property "Description" "Resistor"
-			(at 76.2 123.19 0)
+			(at 73.66 123.19 0)
 			(hide yes)
 			(show_name no)
@@
 		)
 		(property "KiLib_Generator" "SMD_2terminal_chip_molded"
-			(at 76.2 123.19 0)
+			(at 73.66 123.19 0)
 			(hide yes)
 			(show_name no)
@@
 		)
 		(property "LCSC" "C2907034"
-			(at 76.2 123.19 0)
+			(at 73.66 123.19 0)
 			(hide yes)
 			(show_name no)

Commit message: add vio test point
Parts:
- renumbered TP13 to TP14, TP14 to TP15
Changed lines of the file:
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@@
 		(in_pos_files yes)
 		(dnp no)
-		(property "Reference" "TP13"
+		(property "Reference" "TP14"
 			(at 52.07 57.6579 0)
 			(show_name no)
@@
 			(project "syzygy-octosdi"
 				(path "/cb0cdcc9-6b9b-4b74-8146-9043de7999b1/731e7cbd-3c26-4319-8367-0b2702130274"
-					(reference "TP13")
+					(reference "TP14")
 					(unit 1)
 				)
@@
 		(dnp no)
 		(fields_autoplaced yes)
-		(property "Reference" "TP14"
+		(property "Reference" "TP15"
 			(at 60.96 57.6579 0)
 			(show_name no)
@@
 			(project "syzygy-octosdi"
 				(path "/cb0cdcc9-6b9b-4b74-8146-9043de7999b1/731e7cbd-3c26-4319-8367-0b2702130274"
-					(reference "TP14")
-					(unit 1)
-				)
+					(reference "TP15")
+					(unit 1)
+				)

Commit message: sku and led resistor updates following review
Parts:
- D10, D11: LCSC (none) -> C965804
- D12: LCSC (none) -> C965800
- J9: now not fitted
- R78, R79: value 4k7 -> 2k2; LCSC C2907034 -> C2907005
Changed lines of the file:
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@@
+			)
+		)
+		(property "LCSC" "C965800"
+			(at 182.88 130.81 90)
+			(hide yes)
+			(show_name no)
+			(do_not_autoplace no)
+			(effects
+				(font
+					(size 1.27 1.27)
+				)
 			)
 		)
@@
 			)
 		)
+		(property "LCSC" "C965804"
+			(at 73.66 133.35 90)
+			(hide yes)
+			(show_name no)
+			(do_not_autoplace no)
+			(effects
+				(font
+					(size 1.27 1.27)
+				)
+			)
+		)
 		(pin "1"
 		)
@@
 			)
 		)
-		(property "Value" "4k7"
+		(property "Value" "2k2"
 			(at 58.42 124.4599 0)
 			(show_name no)
@@
 			)
 		)
-		(property "LCSC" "C2907034"
+		(property "LCSC" "C2907005"
 			(at 55.88 123.19 0)
 			(hide yes)
@@
 		(on_board yes)
 		(in_pos_files yes)
-		(dnp no)
+		(dnp yes)
 		(fields_autoplaced yes)
 		(property "Reference" "J9"
@@
 			)
 		)
+		(property "LCSC" "C965804"
+			(at 55.88 133.35 90)
+			(hide yes)
+			(show_name no)
+			(do_not_autoplace no)
+			(effects
+				(font
+					(size 1.27 1.27)
+				)
+			)
+		)
 		(pin "1"
 		)
@@
 			)
 		)
-		(property "Value" "4k7"
+		(property "Value" "2k2"
 			(at 76.2 124.4599 0)
 			(show_name no)
@@
 			)
 		)
-		(property "LCSC" "C2907034"
+		(property "LCSC" "C2907005"
 			(at 73.66 123.19 0)
 			(hide yes)
