File: inputs.kicad_sch (KiCad schematic)
At the start: 3 parts, among them U5 PCAL6416AHF

Commit message: split gpio expanders by inputs/outputs instead of quads
Parts:
- C38: renamed from C40; KiLib_Generator (none) -> SMD_2terminal_chip_molded
- C39: renamed from C41; KiLib_Generator (none) -> SMD_2terminal_chip_molded
- U5: KiLib_Generator (none) -> package/no_lead
Connections:
- net SDI Out 1/~{DISABLE} is gone; now on net SDI In 2/BYPASS: U5.5 (P0_4)
- net SDI Out 1/~{EQ_EN} is gone; now on net SDI In 2/MUTE: U5.6 (P0_5)
- net SDI Out 1/~{OSP} is gone; now on net SDI In 2/~{CD}: U5.7 (P0_6)
- net SDI In 2/BYPASS: no longer U5.10 (P1_0)
- net SDI In 2/MUTE: no longer U5.11 (P1_1)
- net SDI In 2/~{CD}: no longer U5.12 (P1_2)
- net SDI Out 1/SD/~{HD}: no longer names the net of U5.4 (P0_3)
- net SDI Out 2/SD/~{HD}: no longer names the net of U5.13 (P1_3)
- net SDI Out 2/~{DISABLE} renamed SDI In 4/BYPASS
- net SDI Out 2/~{EQ_EN} renamed SDI In 4/MUTE
- net SDI Out 2/~{OSP} renamed SDI In 4/~{CD}
- new net SDI In 3/BYPASS: U5.10 (P1_0)
- new net SDI In 3/MUTE: U5.11 (P1_1)
- new net SDI In 3/~{CD}: U5.12 (P1_2)
- no-connect marks 2 -> 4
Other:
- removed sheet SDI Out 1
- removed sheet SDI Out 2
- added sheet SDI In 3 (sdi_in.kicad_sch)
- added sheet SDI In 4 (sdi_in.kicad_sch)

Commit message: add power led and test points
Parts:
- added TP10, TP8, TP9: TestPoint, TestPoint:TestPoint_Pad_D1.0mm, symbol Connector:TestPoint
- renumbered C38 to C40, C39 to C41
Connections:
- net SDI In 1/BYPASS: now also TP8.1
- net SDI In 1/MUTE: now also TP9.1
- net SDI In 1/~{CD}: now also TP10.1

Commit message: check against jlcpcb capabilities
Parts:
- TP10, TP8, TP9: now left out of the parts list
Changed lines of the file:
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@@
 		(body_style 1)
 		(exclude_from_sim no)
-		(in_bom yes)
+		(in_bom no)
 		(on_board yes)
 		(in_pos_files yes)
@@
 		(body_style 1)
 		(exclude_from_sim no)
-		(in_bom yes)
+		(in_bom no)
 		(on_board yes)
 		(in_pos_files yes)
@@
 		(body_style 1)
 		(exclude_from_sim no)
-		(in_bom yes)
-		(on_board yes)
-		(in_pos_files yes)
+		(in_bom no)
+		(on_board yes)
+		(in_pos_files yes)

Commit message: add some larger bypass caps to the cable drivers
Parts:
- renumbered C40 to C41, C41 to C42
Changed lines of the file:
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@@
 		(dnp no)
 		(fields_autoplaced yes)
-		(property "Reference" "#PWR057"
+		(property "Reference" "#PWR059"
 			(at 83.82 66.04 0)
 			(hide yes)
@@
 			(project "syzygy-octosdi"
 				(path "/cb0cdcc9-6b9b-4b74-8146-9043de7999b1/86247bb6-a200-4434-96fd-e477d61cd494"
-					(reference "#PWR057")
+					(reference "#PWR059")
 					(unit 1)
 				)
@@
 		(dnp no)
 		(fields_autoplaced yes)
-		(property "Reference" "#PWR055"
+		(property "Reference" "#PWR057"
 			(at 48.26 114.3 0)
 			(hide yes)
@@
 			(project "syzygy-octosdi"
 				(path "/cb0cdcc9-6b9b-4b74-8146-9043de7999b1/86247bb6-a200-4434-96fd-e477d61cd494"
-					(reference "#PWR055")
+					(reference "#PWR057")
 					(unit 1)
 				)
@@
 		(dnp no)
 		(fields_autoplaced yes)
-		(property "Reference" "#PWR056"
+		(property "Reference" "#PWR058"
 			(at 80.01 124.46 0)
 			(hide yes)
@@
 			(project "syzygy-octosdi"
 				(path "/cb0cdcc9-6b9b-4b74-8146-9043de7999b1/86247bb6-a200-4434-96fd-e477d61cd494"
-					(reference "#PWR056")
+					(reference "#PWR058")
 					(unit 1)
 				)
@@
 		(dnp no)
 		(fields_autoplaced yes)
-		(property "Reference" "C40"
+		(property "Reference" "C41"
 			(at 39.37 101.5999 0)
 			(show_name no)
@@
 			(project "syzygy-octosdi"
 				(path "/cb0cdcc9-6b9b-4b74-8146-9043de7999b1/86247bb6-a200-4434-96fd-e477d61cd494"
-					(reference "C40")
+					(reference "C41")
 					(unit 1)
 				)
@@
 		(dnp no)
 		(fields_autoplaced yes)
-		(property "Reference" "C41"
+		(property "Reference" "C42"
 			(at 52.07 101.5999 0)
 			(show_name no)
@@
 			(project "syzygy-octosdi"
 				(path "/cb0cdcc9-6b9b-4b74-8146-9043de7999b1/86247bb6-a200-4434-96fd-e477d61cd494"
-					(reference "C41")
+					(reference "C42")
 					(unit 1)
 				)
@@
 		(dnp no)
 		(fields_autoplaced yes)
-		(property "Reference" "#PWR054"
+		(property "Reference" "#PWR056"
 			(at 48.26 101.6 0)
 			(hide yes)
@@
 			(project "syzygy-octosdi"
 				(path "/cb0cdcc9-6b9b-4b74-8146-9043de7999b1/86247bb6-a200-4434-96fd-e477d61cd494"
-					(reference "#PWR054")
+					(reference "#PWR056")
 					(unit 1)
 				)
@@
 		(dnp no)
 		(fields_autoplaced yes)
-		(property "Reference" "#PWR053"
+		(property "Reference" "#PWR055"
 			(at 35.56 114.3 0)
 			(hide yes)
@@
 			(project "syzygy-octosdi"
 				(path "/cb0cdcc9-6b9b-4b74-8146-9043de7999b1/86247bb6-a200-4434-96fd-e477d61cd494"
-					(reference "#PWR053")
-					(unit 1)
-				)
+					(reference "#PWR055")
+					(unit 1)
+				)

Commit message: specify skus for parts
Parts:
- C41, C42: LCSC (none) -> C1525
- U5: LCSC (none) -> C2652287
Changed lines of the file:
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@@
+			)
+		)
+		(property "LCSC" "C1525"
+			(at 35.56 102.87 0)
+			(hide yes)
+			(show_name no)
+			(do_not_autoplace no)
+			(effects
+				(font
+					(size 1.27 1.27)
+				)
 			)
 		)
@@
 			)
 		)
+		(property "LCSC" "C1525"
+			(at 48.26 102.87 0)
+			(hide yes)
+			(show_name no)
+			(do_not_autoplace no)
+			(effects
+				(font
+					(size 1.27 1.27)
+				)
+			)
+		)
 		(pin "1"
 		)
@@
 			(at 81.28 90.17 0)
 			(hide yes)
+			(show_name no)
+			(do_not_autoplace no)
+			(effects
+				(font
+					(size 1.27 1.27)
+				)
+			)
+		)
+		(property "LCSC" "C2652287"
+			(at 81.28 90.17 0)
+			(hide yes)

Commit message: add vio test point
Parts:
- renumbered TP9 to TP10, TP10 to TP11, TP8 to TP9
Changed lines of the file:
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@@
 		(in_pos_files yes)
 		(dnp no)
-		(property "Reference" "TP9"
+		(property "Reference" "TP10"
 			(at 111.76 44.958 0)
 			(show_name no)
@@
 			(project "syzygy-octosdi"
 				(path "/cb0cdcc9-6b9b-4b74-8146-9043de7999b1/86247bb6-a200-4434-96fd-e477d61cd494"
-					(reference "TP9")
+					(reference "TP10")
 					(unit 1)
 				)
@@
 		(in_pos_files yes)
 		(dnp no)
-		(property "Reference" "TP8"
+		(property "Reference" "TP9"
 			(at 102.616 54.61 0)
 			(show_name no)
@@
 			(project "syzygy-octosdi"
 				(path "/cb0cdcc9-6b9b-4b74-8146-9043de7999b1/86247bb6-a200-4434-96fd-e477d61cd494"
-					(reference "TP8")
+					(reference "TP9")
 					(unit 1)
 				)
@@
 		(in_pos_files yes)
 		(dnp no)
-		(property "Reference" "TP10"
+		(property "Reference" "TP11"
 			(at 118.11 50.038 0)
 			(show_name no)
@@
 			(project "syzygy-octosdi"
 				(path "/cb0cdcc9-6b9b-4b74-8146-9043de7999b1/86247bb6-a200-4434-96fd-e477d61cd494"
-					(reference "TP10")
-					(unit 1)
-				)
+					(reference "TP11")
+					(unit 1)
+				)
