File: outputs.kicad_sch (KiCad schematic)
At the start: 3 parts, among them U6 PCAL6416AHF

Commit message: fixes following review and more mounting holes
Changed lines of the file:
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@@
 			)
 		)
-		(pin "~{OSP}" input
+		(pin "~{OSP}" output
 			(at 119.38 125.73 180)
 			(effects
@@
 			)
 		)
-		(pin "~{OSP}" input
+		(pin "~{OSP}" output
 			(at 119.38 87.63 180)
 			(effects
@@
 			)
 		)
-		(pin "~{OSP}" input
+		(pin "~{OSP}" output
 			(at 119.38 68.58 180)
 			(effects
@@
 			)
 		)
-		(pin "~{OSP}" input
+		(pin "~{OSP}" output
 			(at 119.38 106.68 180)
 			(effects

Commit message: add power led and test points
Parts:
- added TP11, TP12: TestPoint, TestPoint:TestPoint_Pad_D1.0mm, symbol Connector:TestPoint
- renumbered C40 to C42, C41 to C43
Connections:
- net SDI Out 1/~{DISABLE}: now also TP11.1
- net SDI Out 1/~{OSP}: now also TP12.1

Commit message: check against jlcpcb capabilities
Parts:
- TP11, TP12: now left out of the parts list
Changed lines of the file:
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@@
 		(body_style 1)
 		(exclude_from_sim no)
-		(in_bom yes)
+		(in_bom no)
 		(on_board yes)
 		(in_pos_files yes)
@@
 		(body_style 1)
 		(exclude_from_sim no)
-		(in_bom yes)
+		(in_bom no)
 		(on_board yes)
 		(in_pos_files yes)

Commit message: add some larger bypass caps to the cable drivers
Parts:
- renumbered C42 to C43, C43 to C44
Changed lines of the file:
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@@
 		(dnp no)
 		(fields_autoplaced yes)
-		(property "Reference" "#PWR062"
+		(property "Reference" "#PWR064"
 			(at 83.82 66.04 0)
 			(hide yes)
@@
 			(project "syzygy-octosdi"
 				(path "/cb0cdcc9-6b9b-4b74-8146-9043de7999b1/7952d4e7-438b-4019-af07-2f77390b2cbe"
-					(reference "#PWR062")
+					(reference "#PWR064")
 					(unit 1)
 				)
@@
 		(dnp no)
 		(fields_autoplaced yes)
-		(property "Reference" "#PWR061"
+		(property "Reference" "#PWR063"
 			(at 80.01 124.46 0)
 			(hide yes)
@@
 			(project "syzygy-octosdi"
 				(path "/cb0cdcc9-6b9b-4b74-8146-9043de7999b1/7952d4e7-438b-4019-af07-2f77390b2cbe"
-					(reference "#PWR061")
+					(reference "#PWR063")
 					(unit 1)
 				)
@@
 		(dnp no)
 		(fields_autoplaced yes)
-		(property "Reference" "#PWR058"
+		(property "Reference" "#PWR060"
 			(at 35.56 114.3 0)
 			(hide yes)
@@
 			(project "syzygy-octosdi"
 				(path "/cb0cdcc9-6b9b-4b74-8146-9043de7999b1/7952d4e7-438b-4019-af07-2f77390b2cbe"
-					(reference "#PWR058")
+					(reference "#PWR060")
 					(unit 1)
 				)
@@
 		(dnp no)
 		(fields_autoplaced yes)
-		(property "Reference" "#PWR059"
+		(property "Reference" "#PWR061"
 			(at 48.26 101.6 0)
 			(hide yes)
@@
 			(project "syzygy-octosdi"
 				(path "/cb0cdcc9-6b9b-4b74-8146-9043de7999b1/7952d4e7-438b-4019-af07-2f77390b2cbe"
-					(reference "#PWR059")
+					(reference "#PWR061")
 					(unit 1)
 				)
@@
 		(dnp no)
 		(fields_autoplaced yes)
-		(property "Reference" "C42"
+		(property "Reference" "C43"
 			(at 39.37 101.5999 0)
 			(show_name no)
@@
 			(project "syzygy-octosdi"
 				(path "/cb0cdcc9-6b9b-4b74-8146-9043de7999b1/7952d4e7-438b-4019-af07-2f77390b2cbe"
-					(reference "C42")
+					(reference "C43")
 					(unit 1)
 				)
@@
 		(dnp no)
 		(fields_autoplaced yes)
-		(property "Reference" "C43"
+		(property "Reference" "C44"
 			(at 52.07 101.5999 0)
 			(show_name no)
@@
 			(project "syzygy-octosdi"
 				(path "/cb0cdcc9-6b9b-4b74-8146-9043de7999b1/7952d4e7-438b-4019-af07-2f77390b2cbe"
-					(reference "C43")
+					(reference "C44")
 					(unit 1)
 				)
@@
 		(dnp no)
 		(fields_autoplaced yes)
-		(property "Reference" "#PWR060"
+		(property "Reference" "#PWR062"
 			(at 48.26 114.3 0)
 			(hide yes)
@@
 			(project "syzygy-octosdi"
 				(path "/cb0cdcc9-6b9b-4b74-8146-9043de7999b1/7952d4e7-438b-4019-af07-2f77390b2cbe"
-					(reference "#PWR060")
-					(unit 1)
-				)
+					(reference "#PWR062")
+					(unit 1)
+				)

Commit message: specify skus for parts
Parts:
- C43, C44: LCSC (none) -> C1525
- U6: LCSC (none) -> C2652287
Changed lines of the file:
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@@
+			)
+		)
+		(property "LCSC" "C2652287"
+			(at 81.28 90.17 0)
+			(hide yes)
+			(show_name no)
+			(do_not_autoplace no)
+			(effects
+				(font
+					(size 1.27 1.27)
+				)
 			)
 		)
@@
 			)
 		)
+		(property "LCSC" "C1525"
+			(at 35.56 102.87 0)
+			(hide yes)
+			(show_name no)
+			(do_not_autoplace no)
+			(effects
+				(font
+					(size 1.27 1.27)
+				)
+			)
+		)
 		(pin "1"
 		)
@@
 			(at 48.26 102.87 0)
 			(hide yes)
+			(show_name no)
+			(do_not_autoplace no)
+			(effects
+				(font
+					(size 1.27 1.27)
+				)
+			)
+		)
+		(property "LCSC" "C1525"
+			(at 48.26 102.87 0)
+			(hide yes)

Commit message: add vio test point
Parts:
- renumbered TP11 to TP12, TP12 to TP13
Changed lines of the file:
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@@
 		(in_pos_files yes)
 		(dnp no)
-		(property "Reference" "TP11"
+		(property "Reference" "TP12"
 			(at 107.188 54.102 0)
 			(show_name no)
@@
 			(project "syzygy-octosdi"
 				(path "/cb0cdcc9-6b9b-4b74-8146-9043de7999b1/7952d4e7-438b-4019-af07-2f77390b2cbe"
-					(reference "TP11")
+					(reference "TP12")
 					(unit 1)
 				)
@@
 		(in_pos_files yes)
 		(dnp no)
-		(property "Reference" "TP12"
+		(property "Reference" "TP13"
 			(at 119.38 48.768 0)
 			(show_name no)
@@
 			(project "syzygy-octosdi"
 				(path "/cb0cdcc9-6b9b-4b74-8146-9043de7999b1/7952d4e7-438b-4019-af07-2f77390b2cbe"
-					(reference "TP12")
+					(reference "TP13")
 					(unit 1)
 				)
