File: sdi_out.kicad_sch (KiCad schematic)
At the start: 25 parts, among them J5 Conn_Coaxial, U7 GS2988-INE3

Commit message: add power led and test points
Parts:
- renumbered C42 to C44, C43 to C45, C44 to C46, C45 to C47, C46 to C48, C47 to C49, C48 to C50, C49 to C51, C50 to C52, C51 to C53, D5 to D6, R33 to R34, R34 to R35, R35 to R36, R36 to R37, R37 to R38, R38 to R39, R39 to R40, R40 to R41, R41 to R42, R42 to R43, R43 to R44

Commit message: check against jlcpcb capabilities
Parts:
- J5: value Conn_Coaxial -> Conn_BNC
Changed lines of the file:
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@@
 			)
 		)
-		(property "Value" "Conn_Coaxial"
+		(property "Value" "Conn_BNC"
 			(at 215.9 86.6531 0)
 			(show_name no)

Commit message: add some larger bypass caps to the cable drivers
Parts:
- renumbered C44 to C45, C45 to C46, C46 to C47, C47 to C48, C48 to C49, C49 to C50, C50 to C51, C51 to C52, C52 to C53, C53 to C54

Commit message: specify skus for parts
Parts:
- C45, C46, C51, C52: LCSC (none) -> C15195
- C47, C48, C50, C54: LCSC (none) -> C69335
- C49: LCSC (none) -> C1525
- L5: LCSC (none) -> C3223990
- R36: LCSC (none) -> C21190
- R37: LCSC (none) -> C118388
- R38, R39, R42: LCSC (none) -> C25804
- R40, R41, R43, R44: LCSC (none) -> C324774
Changed lines of the file:
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@@
 			)
 		)
+		(property "LCSC" "C3223990"
+			(at 182.88 85.09 90)
+			(hide yes)
+			(show_name no)
+			(do_not_autoplace no)
+			(effects
+				(font
+					(size 1.27 1.27)
+				)
+			)
+		)
 		(pin "2"
 		)
@@
 			)
 		)
+		(property "LCSC" "C21190"
+			(at 81.28 154.94 0)
+			(hide yes)
+			(show_name no)
+			(do_not_autoplace no)
+			(effects
+				(font
+					(size 1.27 1.27)
+				)
+			)
+		)
 		(pin "1"
 		)
@@
 			)
 		)
+		(property "LCSC" "C118388"
+			(at 83.82 74.93 0)
+			(hide yes)
+			(show_name no)
+			(do_not_autoplace no)
+			(effects
+				(font
+					(size 1.27 1.27)
+				)
+			)
+		)
 		(pin "1"
 		)
@@
 			)
 		)
+		(property "LCSC" "C15195"
+			(at 38.1 41.91 0)
+			(hide yes)
+			(show_name no)
+			(do_not_autoplace no)
+			(effects
+				(font
+					(size 1.27 1.27)
+				)
+			)
+		)
 		(pin "1"
 		)
@@
 			)
 		)
+		(property "LCSC" "C324774"
+			(at 138.43 69.85 0)
+			(hide yes)
+			(show_name no)
+			(do_not_autoplace no)
+			(effects
+				(font
+					(size 1.27 1.27)
+				)
+			)
+		)
 		(pin "2"
 		)
@@
 			)
 		)
+		(property "LCSC" "C324774"
+			(at 182.88 77.47 90)
+			(hide yes)
+			(show_name no)
+			(do_not_autoplace no)
+			(effects
+				(font
+					(size 1.27 1.27)
+				)
+			)
+		)
 		(pin "2"
 		)
@@
 			)
 		)
+		(property "LCSC" "C15195"
+			(at 49.53 41.91 0)
+			(hide yes)
+			(show_name no)
+			(do_not_autoplace no)
+			(effects
+				(font
+					(size 1.27 1.27)
+				)
+			)
+		)
 		(pin "1"
 		)
@@
 			)
 		)
+		(property "LCSC" "C324774"
+			(at 139.7 104.14 0)
+			(hide yes)
+			(show_name no)
+			(do_not_autoplace no)
+			(effects
+				(font
+					(size 1.27 1.27)
+				)
+			)
+		)
 		(pin "2"
 		)
@@
 			)
 		)
+		(property "LCSC" "C69335"
+			(at 198.12 85.09 90)
+			(hide yes)
+			(show_name no)
+			(do_not_autoplace no)
+			(effects
+				(font
+					(size 1.27 1.27)
+				)
+			)
+		)
 		(pin "2"
 		)
@@
 			)
 		)
+		(property "LCSC" "C69335"
+			(at 50.8 78.74 90)
+			(hide yes)
+			(show_name no)
+			(do_not_autoplace no)
+			(effects
+				(font
+					(size 1.27 1.27)
+				)
+			)
+		)
 		(pin "2"
 		)
@@
 			)
 		)
+		(property "LCSC" "C1525"
+			(at 68.58 87.63 90)
+			(hide yes)
+			(show_name no)
+			(do_not_autoplace no)
+			(effects
+				(font
+					(size 1.27 1.27)
+				)
+			)
+		)
 		(pin "1"
 		)
@@
 			)
 		)
+		(property "LCSC" "C25804"
+			(at 124.46 157.48 0)
+			(hide yes)
+			(show_name no)
+			(do_not_autoplace no)
+			(effects
+				(font
+					(size 1.27 1.27)
+				)
+			)
+		)
 		(pin "1"
 		)
@@
 			)
 		)
+		(property "LCSC" "C15195"
+			(at 165.1 68.58 0)
+			(hide yes)
+			(show_name no)
+			(do_not_autoplace no)
+			(effects
+				(font
+					(size 1.27 1.27)
+				)
+			)
+		)
 		(pin "2"
 		)
@@
 			)
 		)
+		(property "LCSC" "C69335"
+			(at 50.8 96.52 90)
+			(hide yes)
+			(show_name no)
+			(do_not_autoplace no)
+			(effects
+				(font
+					(size 1.27 1.27)
+				)
+			)
+		)
 		(pin "2"
 		)
@@
 			)
 		)
+		(property "LCSC" "C25804"
+			(at 140.97 157.48 0)
+			(hide yes)
+			(show_name no)
+			(do_not_autoplace no)
+			(effects
+				(font
+					(size 1.27 1.27)
+				)
+			)
+		)
 		(pin "1"
 		)
@@
 			)
 		)
+		(property "LCSC" "C25804"
+			(at 107.95 157.48 0)
+			(hide yes)
+			(show_name no)
+			(do_not_autoplace no)
+			(effects
+				(font
+					(size 1.27 1.27)
+				)
+			)
+		)
 		(pin "1"
 		)
@@
 			)
 		)
+		(property "LCSC" "C324774"
+			(at 158.75 69.85 0)
+			(hide yes)
+			(show_name no)
+			(do_not_autoplace no)
+			(effects
+				(font
+					(size 1.27 1.27)
+				)
+			)
+		)
 		(pin "2"
 		)
@@
 			)
 		)
+		(property "LCSC" "C15195"
+			(at 144.78 68.58 0)
+			(hide yes)
+			(show_name no)
+			(do_not_autoplace no)
+			(effects
+				(font
+					(size 1.27 1.27)
+				)
+			)
+		)
 		(pin "2"
 		)
@@
 			(at 139.7 93.98 0)
 			(hide yes)
+			(show_name no)
+			(do_not_autoplace no)
+			(effects
+				(font
+					(size 1.27 1.27)
+				)
+			)
+		)
+		(property "LCSC" "C69335"
+			(at 139.7 93.98 0)
+			(hide yes)

Commit message: specify led colours
Parts:
- D6: value LED -> LED Green
Other:
- moved on the sheet: D6, R36
Changed lines of the file:
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@@
 	(text_box "Output Active"
 		(exclude_from_sim no)
-		(at 58.42 138.43 0)
-		(size 33.02 36.83)
+		(at 55.88 138.43 0)
+		(size 37.465 36.83)
 		(margins 0.9525 0.9525 0.9525 0.9525)
 		(stroke
@@
 	(wire
 		(pts
-			(xy 81.28 171.45) (xy 81.28 168.91)
+			(xy 78.74 171.45) (xy 78.74 168.91)
 		)
 		(stroke
@@
 	(wire
 		(pts
-			(xy 81.28 148.59) (xy 81.28 151.13)
+			(xy 78.74 148.59) (xy 78.74 151.13)
 		)
 		(stroke
@@
 	(wire
 		(pts
-			(xy 78.74 171.45) (xy 81.28 171.45)
+			(xy 76.2 171.45) (xy 78.74 171.45)
 		)
 		(stroke
@@
 	(wire
 		(pts
-			(xy 81.28 158.75) (xy 81.28 161.29)
+			(xy 78.74 158.75) (xy 78.74 161.29)
 		)
 		(stroke
@@
 	(hierarchical_label "~{OSP}"
 		(shape output)
-		(at 78.74 171.45 180)
+		(at 76.2 171.45 180)
 		(effects
 			(font
@@
 	(symbol
 		(lib_id "Device:LED")
-		(at 81.28 165.1 90)
+		(at 78.74 165.1 90)
 		(unit 1)
 		(body_style 1)
@@
 		(fields_autoplaced yes)
 		(property "Reference" "D6"
-			(at 85.09 165.4174 90)
+			(at 82.55 165.4174 90)
 			(show_name no)
 			(do_not_autoplace no)
@@
 			)
 		)
-		(property "Value" "LED"
-			(at 85.09 167.9574 90)
+		(property "Value" "LED Green"
+			(at 82.55 167.9574 90)
 			(show_name no)
 			(do_not_autoplace no)
@@
 		)
 		(property "Footprint" "LED_SMD:LED_0603_1608Metric"
-			(at 81.28 165.1 0)
+			(at 78.74 165.1 0)
 			(hide yes)
 			(show_name no)
@@
 		)
 		(property "Datasheet" ""
-			(at 81.28 165.1 0)
+			(at 78.74 165.1 0)
 			(hide yes)
 			(show_name no)
@@
 		)
 		(property "Description" "Light emitting diode"
-			(at 81.28 165.1 0)
+			(at 78.74 165.1 0)
 			(hide yes)
 			(show_name no)
@@
 		)
 		(property "Sim.Pins" "1=K 2=A"
-			(at 81.28 165.1 0)
+			(at 78.74 165.1 0)
 			(hide yes)
 			(show_name no)
@@
 		)
 		(property "KiLib_Generator" "SMD_2terminal_chip_molded"
-			(at 81.28 165.1 0)
+			(at 78.74 165.1 0)
 			(hide yes)
 			(show_name no)
@@
 	(symbol
 		(lib_id "Device:R")
-		(at 81.28 154.94 0)
+		(at 78.74 154.94 0)
 		(mirror y)
 		(unit 1)
@@
 		(fields_autoplaced yes)
 		(property "Reference" "R36"
-			(at 83.82 153.6699 0)
+			(at 81.28 153.6699 0)
 			(show_name no)
 			(do_not_autoplace no)
@@
 		)
 		(property "Value" "1k"
-			(at 83.82 156.2099 0)
+			(at 81.28 156.2099 0)
 			(show_name no)
 			(do_not_autoplace no)
@@
 		)
 		(property "Footprint" "Resistor_SMD:R_0603_1608Metric"
-			(at 83.058 154.94 90)
+			(at 80.518 154.94 90)
 			(hide yes)
 			(show_name no)
@@
 		)
 		(property "Datasheet" ""
-			(at 81.28 154.94 0)
+			(at 78.74 154.94 0)
 			(hide yes)
 			(show_name no)
@@
 		)
 		(property "Description" "Resistor"
-			(at 81.28 154.94 0)
+			(at 78.74 154.94 0)
 			(hide yes)
 			(show_name no)
@@
 		)
 		(property "KiLib_Generator" "SMD_2terminal_chip_molded"
-			(at 81.28 154.94 0)
+			(at 78.74 154.94 0)
 			(hide yes)
 			(show_name no)
@@
 		)
 		(property "LCSC" "C21190"
-			(at 81.28 154.94 0)
+			(at 78.74 154.94 0)
 			(hide yes)
 			(show_name no)
@@
 	(symbol
 		(lib_id "power:+3V3")
-		(at 81.28 148.59 0)
+		(at 78.74 148.59 0)
 		(unit 1)
 		(body_style 1)
@@
 		(fields_autoplaced yes)
 		(property "Reference" "#PWR068"
-			(at 81.28 152.4 0)
+			(at 78.74 152.4 0)
 			(hide yes)
 			(show_name no)
@@
 		)
 		(property "Value" "+3V3"
-			(at 81.28 143.51 0)
+			(at 78.74 143.51 0)
 			(show_name no)
 			(do_not_autoplace no)
@@
 		)
 		(property "Footprint" ""
-			(at 81.28 148.59 0)
+			(at 78.74 148.59 0)
 			(hide yes)
 			(show_name no)
@@
 		)
 		(property "Datasheet" ""
-			(at 81.28 148.59 0)
+			(at 78.74 148.59 0)
 			(hide yes)
 			(show_name no)
@@
 		)
 		(property "Description" "Power symbol creates a global label with name \"+3V3\""
-			(at 81.28 148.59 0)
+			(at 78.74 148.59 0)
 			(hide yes)
 			(show_name no)

Commit message: sku and led resistor updates following review
Parts:
- D6: LCSC (none) -> C965804
Changed lines of the file:
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@@
+			)
+		)
+		(property "LCSC" "C965804"
+			(at 78.74 165.1 90)
+			(hide yes)
+			(show_name no)
+			(do_not_autoplace no)
+			(effects
+				(font
+					(size 1.27 1.27)
+				)
 			)
 		)
